File: MMS3_hat_protcol_board_basic.kicad_sch (KiCad schematic)
At the start: 16 parts, among them J11 Conn_01x04_Pin, J4 Conn_01x04_Pin, J7 Conn_01x06_Pin, U3 AMS1117

Commit message: updated routing, removed megamind
Parts:
- removed PN1: ~, PCM_JLCPCB:Part_Num_JLCPCB, symbol PCM_JLCPCB-Manufacturing:Part Number, PCM_JLCPCB, 0.8x0.15mm
- H7, H8, H9: value ~ -> (none)
